File: Amiga_Ashcom_512Kb.kicad_sch (KiCad schematic)
At the start: 22 parts, among them J1 Amiga expansion port, U1 74LS00, U2 xx4256, U3 xx4256, U4 xx4256, U5 xx4256, U6 M6242B, Y1 Crystal

Commit message: Annotated the schematic to match the PCB, and added experimental gerbers.
Parts:
- C1, C3, C4, C5: footprint (none) -> Capacitor_THT:C_Axial_L5.1mm_D3.1mm_P7.50mm_Horizontal
- C7, C8: value 100nF -> 22pF; footprint (none) -> Capacitor_THT:C_Disc_D3.0mm_W1.6mm_P2.50mm
- C9: footprint (none) -> Capacitor_THT:C_Disc_D3.0mm_W1.6mm_P2.50mm
- J1: footprint (none) -> Connector_PinSocket_2.54mm:PinSocket_2x28_P2.54mm_Horizontal
- R1: renamed from R2; footprint (none) -> Resistor_THT:R_Axial_DIN0204_L3.6mm_D1.6mm_P7.62mm_Horizontal
- R2: footprint (none) -> Resistor_THT:R_Axial_DIN0204_L3.6mm_D1.6mm_P7.62mm_Horizontal
- S1: footprint (none) -> footprints:780565
- U1: renamed from U6; footprint (none) -> Package_DIP:DIP-14_W7.62mm_LongPads
- U1: footprint (none) -> Package_DIP:DIP-14_W7.62mm_LongPads
- U2, U3, U4, U5: footprint (none) -> Package_DIP:DIP-20_W7.62mm_LongPads
- U6: footprint (none) -> Package_DIP:DIP-18_W7.62mm_LongPads
- Y1: footprint (none) -> Crystal:Crystal_C26-LF_D2.1mm_L6.5mm_Vertical
- renumbered RN2 to RN3
Connections:
- net GND: now also U2.5 (NC), U3.5 (NC), U4.5 (NC), U5.5 (NC)
Other:
- title: (none) -> Ashcom 512Kb expansion card for an Amiga 500

Commit message: Fix R1/R2 references and values, change C9 to 100nF
Parts:
- renumbered R2 to R1, R1 to R2
Changed lines of the file:
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@@
 		(on_board yes)
 		(dnp no)
-		(property "Reference" "R2"
+		(property "Reference" "R1"
 			(at 91.44 85.598 90)
 			(effects
@@
 			(project ""
 				(path "/aa78249d-245e-4f40-822e-739672b24332"
-					(reference "R2")
+					(reference "R1")
 					(unit 1)
 				)
@@
 		(dnp no)
 		(fields_autoplaced yes)
-		(property "Reference" "R1"
+		(property "Reference" "R2"
 			(at 29.21 147.3199 0)
 			(effects
@@
 			(project ""
 				(path "/aa78249d-245e-4f40-822e-739672b24332"
-					(reference "R1")
-					(unit 1)
-				)
+					(reference "R2")
+					(unit 1)
+				)
